Commit message: reachy_mini: hardware sign table in ROBOT.md, antenna values = plain daemon values everywhere, daemon URDF confirmed identical to vendor
Co-Authored-By: Claude Fable 5 <noreply@anthropic.com>
Claude-Session: https://claude.ai/code/session_01XLrich3HFtpCda854Pq99i

File: robots/reachy_mini/urdf/reachy_mini.urdf (robot description, URDF)
Before this commit: robot reachy_mini, 11 links, 10 joints
Joints:
- joint antenna_left: axis 0 0 -1 -> 0 0 1
- joint antenna_right: axis 0 0 -1 -> 0 0 1
